Commit message: Organice el archivo urdf

File: install/manipulator_description/share/manipulator_description/urdf/manipulator.urdf.xacro (robot description, xacro)
@@ -1,4 +1,7 @@
 <?xml version="1.0"?>
 <robot xmlns:xacro="http://www.ros.org/wiki/xacro"  name="manipulator">
+  <xacro:property name="PI" value="3.14159"/>
+  <xacro:property name="effort" value="300.0"/>
+  <xacro:property name="velocity" value="3.0"/>
   <link name="base_footprint"/>
   <joint name="base_joint" type="fixed">
@@ -7,275 +10,150 @@
     <origin xyz="0 0 0" rpy="0 0 0"/>
   </joint>
-  <link
-    name="base_link">
+  <link name="base_link">
     <inertial>
-      <origin
-        xyz="7.2577E-09 -0.031297 0.093199"
-        rpy="0 0 0" />
-      <mass
-        value="20.05" />
-      <inertia
-        ixx="0.42459"
-        ixy="2.2307E-08"
-        ixz="5.8415E-08"
-        iyy="0.34019"
-        iyz="0.040988"
-        izz="0.49886" />
+      <origin xyz="7.2577E-09 -0.031297 0.093199" rpy="0 0 0"/>
+      <mass value="20.05"/>
+      <inertia ixx="0.42459" ixy="2.2307E-08" ixz="5.8415E-08" iyy="0.34019" iyz="0.040988" izz="0.49886"/>
     </inertial>
     <visual>
-      <origin
-        xyz="0 0 0"
-        rpy="0 0 0" />
+      <origin xyz="0 0 0" rpy="0 0 0"/>
       <geometry>
-        <mesh
-          filename="package://manipulator_description/meshes/base_link.STL" />
+        <mesh filename="package://manipulator_description/meshes/base_link.STL"/>
+      </geometry>
+      <material name="">
+        <!-- <color rgba="0.79216 0.81961 0.93333 1" /> -->
+      </material>
+    </visual>
+    <collision>
+      <origin xyz="0 0 0" rpy="0 0 0"/>
+      <geometry>
+        <mesh filename="package://manipulator_description/meshes/base_link.STL"/>
+      </geometry>
+    </collision>
+  </link>
+  <link name="link_1">
+    <inertial>
+      <origin xyz="-1.5626E-10 0.21308 1.1102E-16" rpy="0 0 0"/>
+      <mass value="14.515"/>
+      <inertia ixx="0.28139" ixy="-1.2685E-09" ixz="1.2578E-09" iyy="0.10949" iyz="-1.4778E-17" izz="0.30806"/>
+    </inertial>
+    <visual>
+      <origin xyz="0 0 0" rpy="0 0 0"/>
+      <geometry>
+        <mesh filename="package://manipulator_description/meshes/link_1.STL"/>
       </geometry>
       <material
         name="">
-        <color
-          rgba="0.79216 0.81961 0.93333 1" />
+        <!-- <color rgba="0.79216 0.81961 0.93333 1" /> -->
       </material>
     </visual>
     <collision>
-      <origin
-        xyz="0 0 0"
-        rpy="0 0 0" />
+      <origin xyz="0 0 0" rpy="0 0 0"/>
       <geometry>
-        <mesh
-          filename="package://manipulator_description/meshes/base_link.STL" />
+        <mesh filename="package://manipulator_description/meshes/link_1.STL"/>
       </geometry>
     </collision>
   </link>
-  <link
-    name="link_1">
+  <joint name="joint_1" type="revolute">
+    <origin xyz="0 0 0.16" rpy="1.5708 0 0"/>
+    <parent link="base_link"/>
+    <child link="link_1" />
+    <axis xyz="0 1 0" />
+    <!-- <limit lower="0" upper="3.142" effort="300" velocity="3"/> -->
+    <limit lower="-${PI/2}" upper="${PI/2}" effort="${effort}" velocity="${velocity}"/>
+  </joint>
+  <link name="link_2">
     <inertial>
       <origin
-        xyz="-1.5626E-10 0.21308 1.1102E-16"
-        rpy="0 0 0" />
-      <mass
-        value="14.515" />
-      <inertia
-        ixx="0.28139"
-        ixy="-1.2685E-09"
-        ixz="1.2578E-09"
-        iyy="0.10949"
-        iyz="-1.4778E-17"
-        izz="0.30806" />
+        xyz="7.9787E-10 2.6404E-11 -0.19156" rpy="0 0 0"/>
+      <mass value="15.461"/>
+      <inertia ixx="0.71519" ixy="-2.5469E-10" ixz="2.0918E-09" iyy="0.62073" iyz="9.6415E-11" izz="0.15696"/>
     </inertial>
     <visual>
-      <origin
-        xyz="0 0 0"
-        rpy="0 0 0" />
+      <origin xyz="0 0 0" rpy="0 0 0"/>
       <geometry>
-        <mesh
-          filename="package://manipulator_description/meshes/link_1.STL" />
+        <mesh filename="package://manipulator_description/meshes/link_2.STL"/>
       </geometry>
       <material
         name="">
-        <color
-          rgba="0.79216 0.81961 0.93333 1" />
+        <!-- <color rgba="0.79216 0.81961 0.93333 1" /> -->
       </material>
     </visual>
     <collision>
-      <origin
-        xyz="0 0 0"
-        rpy="0 0 0" />
+      <origin xyz="0 0 0" rpy="0 0 0"/>
       <geometry>
-        <mesh
-          filename="package://manipulator_description/meshes/link_1.STL" />
+        <mesh filename="package://manipulator_description/meshes/link_2.STL"/>
       </geometry>
     </collision>
   </link>
-  <joint
-    name="joint_1"
-    type="revolute">
-    <origin
-      xyz="0 0 0.16"
-      rpy="1.5708 0 0" />
-    <parent
-      link="base_link" />
-    <child
-      link="link_1" />
-    <axis
-      xyz="0 1 0" />
-    <limit
-      lower="0"
-      upper="3.142"
-      effort="300"
-      velocity="3" />
+  <joint name="joint_2" type="revolute">
+    <origin xyz="0 0.336 0" rpy="-1.5708 0 3.1243"/>
+    <parent link="link_1"/>
+    <child link="link_2"/>
+    <axis xyz="0 -1 0"/>
+    <!-- <limit lower="-1.57" upper="1.57" effort="200" velocity="3"/> -->
+    <limit lower="-${PI/2}" upper="${PI/2}" effort="${effort}" velocity="${velocity}"/>
   </joint>
-  <link
-    name="link_2">
+  <link name="link_3">
     <inertial>
-      <origin
-        xyz="7.9787E-10 2.6404E-11 -0.19156"
-        rpy="0 0 0" />
-      <mass
-        value="15.461" />
-      <inertia
-        ixx="0.71519"
-        ixy="-2.5469E-10"
-        ixz="2.0918E-09"
-        iyy="0.62073"
-        iyz="9.6415E-11"
-        izz="0.15696" />
+      <origin xyz="0.13619 0.12118 7.1719E-10" rpy="0 0 0"/>
+      <mass value="12.06"/>
+      <inertia ixx="0.075233" ixy="-0.039898" ixz="-2.2298E-10" iyy="0.3384" iyz="-8.9743E-10" izz="0.37074"/>
     </inertial>
     <visual>
-      <origin
-        xyz="0 0 0"
-        rpy="0 0 0" />
+      <origin xyz="0 0 0" rpy="0 0 0"/>
       <geometry>
-        <mesh
-          filename="package://manipulator_description/meshes/link_2.STL" />
+        <mesh filename="package://manipulator_description/meshes/link_3.STL"/>
       </geometry>
       <material
         name="">
-        <color
-          rgba="0.79216 0.81961 0.93333 1" />
+        <!-- <color rgba="0.79216 0.81961 0.93333 1" /> -->
       </material>
     </visual>
     <collision>
-      <origin
-        xyz="0 0 0"
-        rpy="0 0 0" />
+      <origin xyz="0 0 0" rpy="0 0 0"/>
       <geometry>
-        <mesh
-          filename="package://manipulator_description/meshes/link_2.STL" />
+        <mesh filename="package://manipulator_description/meshes/link_3.STL"/>
       </geometry>
     </collision>
   </link>
-  <joint
-    name="joint_2"
-    type="revolute">
-    <origin
-      xyz="0 0.336 0"
-      rpy="-1.5708 0 3.1243" />
-    <parent
-      link="link_1" />
-    <child
-      link="link_2" />
-    <axis
-      xyz="0 -1 0" />
-    <limit
-      lower="-1.57"
-      upper="1.57"
-      effort="200"
-      velocity="3" />
+  <joint name="joint_3" type="revolute">
+    <origin xyz="0 0 -0.5" rpy="-1.5708 0.017244 3.1416"/>
+    <parent link="link_2"/>
+    <child link="link_3"/>
+    <axis xyz="0 0 1"/>
+    <!-- <limit lower="0" upper="3.142" effort="200" velocity="3"/> -->
+    <limit lower="-${PI/2}" upper="${PI/2}" effort="${effort}" velocity="${velocity}"/>
   </joint>
-  <link
-    name="link_3">
+  <link name="link_4">
     <inertial>
-      <origin
-        xyz="0.13619 0.12118 7.1719E-10"
-        rpy="0 0 0" />
-      <mass
-        value="12.06" />
-      <inertia
-        ixx="0.075233"
-        ixy="-0.039898"
-        ixz="-2.2298E-10"
-        iyy="0.3384"
-        iyz="-8.9743E-10"
-        izz="0.37074" />
+      <origin xyz="0.023573 4.3615E-08 -2.3893E-09" rpy="0 0 0"/>
+      <mass value="1.1724"/>
+      <inertia ixx="0.0021334" ixy="-1.5043E-09" ixz="-2.9639E-11" iyy="0.0061469" iyz="-1.2799E-09" izz="0.0066548"/>
     </inertial>
     <visual>
-      <origin
-        xyz="0 0 0"
-        rpy="0 0 0" />
+      <origin xyz="0 0 0" rpy="0 0 0"/>
       <geometry>
-        <mesh
-          filename="package://manipulator_description/meshes/link_3.STL" />
+        <mesh filename="package://manipulator_description/meshes/link_4.STL"/>
       </geometry>
       <material
         name="">
-        <color
-          rgba="0.79216 0.81961 0.93333 1" />
+        <!-- <color rgba="0.79216 0.81961 0.93333 1" /> -->
       </material>
     </visual>
     <collision>
-      <origin
-        xyz="0 0 0"
-        rpy="0 0 0" />
+      <origin xyz="0 0 0" rpy="0 0 0"/>
       <geometry>
-        <mesh
-          filename="package://manipulator_description/meshes/link_3.STL" />
+        <mesh filename="package://manipulator_description/meshes/link_4.STL"/>
       </geometry>
     </collision>
   </link>
-  <joint
-    name="joint_3"
-    type="revolute">
-    <origin
-      xyz="0 0 -0.5"
-      rpy="-1.5708 0.017244 3.1416" />
-    <parent
-      link="link_2" />
-    <child
-      link="link_3" />
-    <axis
-      xyz="0 0 1" />
-    <limit
-      lower="0"
-      upper="3.142"
-      effort="200"
-      velocity="3" />
-  </joint>
-  <link
-    name="link_4">
-    <inertial>
-      <origin
-        xyz="0.023573 4.3615E-08 -2.3893E-09"
-        rpy="0 0 0" />
-      <mass
-        value="1.1724" />
-      <inertia
-        ixx="0.0021334"
-        ixy="-1.5043E-09"
-        ixz="-2.9639E-11"
-        iyy="0.0061469"
-        iyz="-1.2799E-09"
-        izz="0.0066548" />
-    </inertial>
-    <visual>
-      <origin
-        xyz="0 0 0"
-        rpy="0 0 0" />
-      <geometry>
-        <mesh
-          filename="package://manipulator_description/meshes/link_4.STL" />
-      </geometry>
-      <material
-        name="">
-        <color
-          rgba="0.79216 0.81961 0.93333 1" />
-      </material>
-    </visual>
-    <collision>
-      <origin
-        xyz="0 0 0"
-        rpy="0 0 0" />
-      <geometry>
-        <mesh
-          filename="package://manipulator_description/meshes/link_4.STL" />
-      </geometry>
-    </collision>
-  </link>
-  <joint
-    name="joint_4"
-    type="revolute">
-    <origin
-      xyz="0.42746 0.145 0"
-      rpy="0 0 -0.017244" />
-    <parent
-      link="link_3" />
-    <child
-      link="link_4" />
-    <axis
-      xyz="0 0 1" />
-    <limit
-      lower="-3.142"
-      upper="3.142"
-      effort="200"
-      velocity="3" />
+  <joint name="joint_4" type="revolute">
+    <origin xyz="0.42746 0.145 0" rpy="0 0 -0.017244"/>
+    <parent link="link_3"/>
+    <child link="link_4"/>
+    <axis xyz="0 0 1"/>
+    <!-- <limit lower="-3.142" upper="3.142" effort="200" velocity="3"/> -->
+    <limit lower="-${PI/2}" upper="${PI/2}" effort="${effort}" velocity="${velocity}"/>
   </joint>
 </robot>
